File: horangi_grin/pcb/horangi_left.kicad_pcb (KiCad board)
At the start: 2 copper layers, 171.7 x 130.2 mm, 50 parts, among them SW1 Switch, SW10 Switch, SW11 Switch, SW12 Switch, SW13 Switch, SW14 Switch, SW15 Switch, SW16 Switch, SW17 Switch, SW18 Switch, SW19 Switch, SW2 Switch, SW20 Switch, SW21 Switch, SW22 Switch, SW23 Switch, SW24 Switch, SW25 Switch, SW26 Switch, SW27 Switch, SW28 Switch, SW29 Switch, SW3 Switch, SW30 Switch, SW31 Switch, SW32 Switch, SW33 Switch, SW34 Switch, SW35 Switch, SW37 Switch, SW38 Switch, SW39 Switch, SW4 Switch, SW40 Switch, SW41 Switch, SW42 Switch, SW5 Switch, SW6 Switch, SW7 Switch, SW8 Switch, SW9 Switch

Commit message: update horangi
Changed lines of the file:
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@@
       (drillshape 0)
       (scaleselection 1)
-      (outputdirectory "gerber_left/")
+      (outputdirectory "gerber_horangi_left/")
     )
   )
@@
       (effects (font (size 1.27 1.27) (thickness 0.15)))
     )
-    (pad "" np_thru_hole circle (at 0 0 90) (size 7.2 7.2) (drill 7.2) (layers F&B.Cu *.Mask))
+    (pad "" np_thru_hole circle (at 0 0 90) (size 7.5 7.5) (drill 7.5) (layers F&B.Cu *.Mask))
   )
   (footprint "footprints:MX-hotswap-diode-smd" (layer "F.Cu")
@@
       (effects (font (size 1.27 1.27) (thickness 0.15)))
     )
-    (pad "" np_thru_hole circle (at 0 0 90) (size 7.2 7.2) (drill 7.2) (layers F&B.Cu *.Mask))
+    (pad "" np_thru_hole circle (at 0 0 90) (size 7.5 7.5) (drill 7.5) (layers F&B.Cu *.Mask))
   )
   (footprint "footprints:MX-hotswap-diode-smd" (layer "F.Cu")
@@
       (effects (font (size 1.27 1.27) (thickness 0.15)))
     )
-    (pad "" np_thru_hole circle (at 0 0 90) (size 7.2 7.2) (drill 7.2) (layers F&B.Cu *.Mask))
+    (pad "" np_thru_hole circle (at 0 0 90) (size 7.5 7.5) (drill 7.5) (layers F&B.Cu *.Mask))
   )
   (footprint "footprints:MX-hotswap-diode-smd" (layer "F.Cu")
@@
       (effects (font (size 1.27 1.27) (thickness 0.15)))
     )
-    (pad "" np_thru_hole circle (at 0 0 90) (size 7.2 7.2) (drill 7.2) (layers F&B.Cu *.Mask))
+    (pad "" np_thru_hole circle (at 0 0 90) (size 7.5 7.5) (drill 7.5) (layers F&B.Cu *.Mask))
   )
   (footprint "footprints:MX-hotswap-diode-smd" (layer "F.Cu")
