File: horangi_grin/pcb/horangi_right.kicad_pcb (KiCad board)
At the start: 2 copper layers, 171.7 x 130.2 mm, 51 parts, among them SW1 Switch, SW10 Switch, SW11 Switch, SW12 Switch, SW13 Switch, SW14 Switch, SW15 Switch, SW16 Switch, SW17 Switch, SW18 Switch, SW19 Switch, SW2 Switch, SW20 Switch, SW21 Switch, SW22 Switch, SW23 Switch, SW24 Switch, SW25 Switch, SW26 Switch, SW27 Switch, SW28 Switch, SW29 Switch, SW3 Switch, SW30 Switch, SW31 Switch, SW32 Switch, SW33 Switch, SW34 Switch, SW35 Switch, SW36 Switch, SW37 Switch, SW38 Switch, SW39 Switch, SW4 Switch, SW40 Switch, SW41 Switch, SW42 Switch, SW5 Switch, SW6 Switch, SW7 Switch, SW8 Switch, SW9 Switch

Commit message: update horangi
Routing:
- net ROW5: track 173.3 -> 174.6 mm
Changed lines of the file:
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@@
       (drillshape 0)
       (scaleselection 1)
-      (outputdirectory "gerber_right/")
+      (outputdirectory "gerber_horangi_right/")
     )
   )
@@
       (effects (font (size 1.27 1.27) (thickness 0.15)))
     )
-    (pad "" np_thru_hole circle (at 0 0 90) (size 7.2 7.2) (drill 7.2) (layers F&B.Cu *.Mask))
+    (pad "" np_thru_hole circle (at 0 0 90) (size 7.5 7.5) (drill 7.5) (layers F&B.Cu *.Mask))
   )
   (footprint "footprints:MX-hotswap-diode-smd" (layer "F.Cu")
@@
       (effects (font (size 1.27 1.27) (thickness 0.15)))
     )
-    (pad "" np_thru_hole circle (at 0 0 90) (size 7.2 7.2) (drill 7.2) (layers F&B.Cu *.Mask))
+    (pad "" np_thru_hole circle (at 0 0 90) (size 7.5 7.5) (drill 7.5) (layers F&B.Cu *.Mask))
   )
   (footprint "" (layer "F.Cu")
@@
       (effects (font (size 1.27 1.27) (thickness 0.15)))
     )
-    (pad "" np_thru_hole circle (at 0 0 90) (size 7.2 7.2) (drill 7.2) (layers F&B.Cu *.Mask))
+    (pad "" np_thru_hole circle (at 0 0 90) (size 7.5 7.5) (drill 7.5) (layers F&B.Cu *.Mask))
   )
   (footprint "footprints:MX-hotswap-diode-smd_1.25u" (layer "F.Cu")
@@
       (effects (font (size 1.27 1.27) (thickness 0.15)))
     )
-    (pad "" np_thru_hole circle (at 0 0 90) (size 7.2 7.2) (drill 7.2) (layers F&B.Cu *.Mask))
+    (pad "" np_thru_hole circle (at 0 0 90) (size 7.5 7.5) (drill 7.5) (layers F&B.Cu *.Mask))
   )
   (footprint "footprints:MX-hotswap-diode-smd" (layer "F.Cu")
@@
   (segment (start 219.936706 84.517525) (end 219.936706 80.94222) (width 0.25) (layer "F.Cu") (net 23))
   (segment (start 227.309118 118.242525) (end 217.711706 118.242525) (width 0.25) (layer "F.Cu") (net 23))
+  (segment (start 147.045708 153.958736) (end 148.769497 155.682525) (width 0.25) (layer "B.Cu") (net 64))
   (segment (start 123.372997 157.294817) (end 143.709627 157.294817) (width 0.25) (layer "B.Cu") (net 64))
   (segment (start 201.266706 150.775025) (end 220.316706 150.775025) (width 0.25) (layer "B.Cu") (net 64))
   (segment (start 203.634206 134.092525) (end 217.784206 134.092525) (width 0.25) (layer "B.Cu") (net 64))
-  (segment (start 178.253206 154.875035) (end 182.216706 150.911535) (width 0.25) (layer "B.Cu") (net 64))
   (segment (start 217.784206 134.092525) (end 217.784206 148.242525) (width 0.25) (layer "B.Cu") (net 64))
-  (segment (start 182.216706 150.911535) (end 182.216706 150.775025) (width 0.25) (layer "B.Cu") (net 64))
-  (segment (start 147.962007 154.875035) (end 178.253206 154.875035) (width 0.25) (layer "B.Cu") (net 64))
+  (segment (start 148.769497 155.682525) (end 178.511706 155.682525) (width 0.25) (layer "B.Cu") (net 64))
   (segment (start 217.784206 148.242525) (end 220.316706 150.775025) (width 0.25) (layer "B.Cu") (net 64))
   (segment (start 143.709627 157.294817) (end 147.045708 153.958736) (width 0.25) (layer "B.Cu") (net 64))
   (segment (start 182.216706 150.775025) (end 201.266706 150.775025) (width 0.25) (layer "B.Cu") (net 64))
   (segment (start 87.379587 161.151051) (end 88.417168 160.11347) (width 0.25) (layer "B.Cu") (net 64))
+  (segment (start 178.511706 155.682525) (end 182.216706 151.977525) (width 0.25) (layer "B.Cu") (net 64))
   (segment (start 88.417168 160.11347) (end 120.554344 160.11347) (width 0.25) (layer "B.Cu") (net 64))
   (segment (start 120.554344 160.11347) (end 123.372997 157.294817) (width 0.25) (layer "B.Cu") (net 64))
-  (segment (start 147.045708 153.958736) (end 147.962007 154.875035) (width 0.25) (layer "B.Cu") (net 64))
   (segment (start 201.266706 131.725025) (end 203.634206 134.092525) (width 0.25) (layer "B.Cu") (net 64))
+  (segment (start 182.216706 151.977525) (end 182.216706 150.775025) (width 0.25) (layer "B.Cu") (net 64))
   (zone (net 2) (net_name "GND") (layers F&B.Cu) (hatch edge 0.508)
     (connect_pads (clearance 0.508))
